File: schematic/button-board/button-board.kicad_pcb (KiCad board)
At the start: 2 copper layers, 47 parts, among them J10 Conn_01x04_Socket, J11 Conn_01x04_Socket, J12 Conn_01x04_Socket, J13 Conn_01x04_Socket, J14 Conn_01x04_Socket, J16 Screw_Terminal_01x06, J2 Screw_Terminal_01x08, J3 Screw_Terminal_01x08, J7 Conn_01x04_Socket, J8 Conn_01x04_Socket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

Commit message: layout work
Parts:
- removed J12, J13, J14: Conn_01x04_Socket, Connector_JST:JST_XH_B4B-XH-AM_1x04_P2.50mm_Vertical
- removed J16: Screw_Terminal_01x06, TerminalBlock:TerminalBlock_bornier-6_P5.08mm
- removed Q10, Q11, Q12, Q4, Q5, Q6, Q7, Q9: 2N7002, Package_TO_SOT_SMD:SOT-23
- removed R11, R13, R15, R23, R25, R27, R29: 1k, Resistor_SMD:R_0805_2012Metric
- removed R12, R14, R22, R24, R26, R28: 10k, Resistor_SMD:R_0805_2012Metric
- removed R16, R17: 4k7, Resistor_SMD:R_0805_2012Metric
- removed R18, R20: 330R, Resistor_SMD:R_0805_2012Metric
- added J1: ~, SparkFun-Connector:1x04_RA_SMD, F.Cu at (112.5, 125.0)
- added J4: Screw_Terminal_01x04, TerminalBlock_Phoenix:TerminalBlock_Phoenix_MKDS-1,5-4-5.08_1x04_P5.08mm_Horizontal, F.Cu at (139.8, 51.0)
- added J5: Screw_Terminal_01x04, TerminalBlock_Phoenix:TerminalBlock_Phoenix_MKDS-1,5-4-5.08_1x04_P5.08mm_Horizontal, F.Cu at (139.8, 62.1)
- added J6: Screw_Terminal_01x04, TerminalBlock_Phoenix:TerminalBlock_Phoenix_MKDS-1,5-4-5.08_1x04_P5.08mm_Horizontal, F.Cu at (139.8, 73.3)
- added JP4: SolderJumper_3_Bridged123, Jumper:SolderJumper-3_P1.3mm_Bridged123_RoundedPad1.0x1.5mm_NumberLabels, F.Cu at (115.0, 110.5)
- added R1: 4k7, Resistor_SMD:R_0805_2012Metric, F.Cu at (113.5, 115.5)
- added R3: 1k, Resistor_SMD:R_0805_2012Metric, F.Cu at (131.6, 47.0)
- added R4: 1k, Resistor_SMD:R_0805_2012Metric, F.Cu at (131.6, 58.0)
- added R5: 1k, Resistor_SMD:R_0805_2012Metric, F.Cu at (131.6, 69.0)
- added R6: 1k, Resistor_SMD:R_0805_2012Metric, F.Cu at (131.6, 80.0)
- added R7: 1k, Resistor_SMD:R_0805_2012Metric, F.Cu at (131.6, 91.5)
- added U2: ULN2803A, Package_SO:SOP-18_7.495x11.515mm_P1.27mm, F.Cu at (96.7, 90.6)
- C1: value 0.1u -> 47u; footprint Capacitor_SMD:C_0805_2012Metric -> Capacitor_THT:C_Radial_D6.3mm_H11.0mm_P2.50mm
- C2: value 47u -> 0.1u; footprint Capacitor_THT:C_Radial_D6.3mm_H11.0mm_P2.50mm -> Capacitor_SMD:C_0805_2012Metric
- J10, J11, J7, J8, J9: value Conn_01x04_Socket -> Screw_Terminal_01x04; footprint Connector_JST:JST_XH_B4B-XH-AM_1x04_P2.50mm_Vertical -> TerminalBlock_Phoenix:TerminalBlock_Phoenix_MKDS-1,5-4-5.08_1x04_P5.08mm_Horizontal
- J2: value Screw_Terminal_01x08 -> ~; footprint TerminalBlock:TerminalBlock_bornier-8_P5.08mm -> SparkFun-Connector:1x04_RA_SMD
- J3: value Screw_Terminal_01x08 -> Screw_Terminal_01x02; footprint TerminalBlock:TerminalBlock_bornier-8_P5.08mm -> TerminalBlock_Phoenix:TerminalBlock_Phoenix_MKDS-1,5-2-5.08_1x02_P5.08mm_Horizontal
- JP1, JP2, JP3: footprint Jumper:SolderJumper-3_P1.3mm_Bridged12_RoundedPad1.0x1.5mm -> Jumper:SolderJumper-3_P1.3mm_Bridged12_RoundedPad1.0x1.5mm_NumberLabels
- R10, R8: value 10k -> 1k
- R2: value 10k -> 4k7
- moved J7 110.2 mm to (140.0, 84.4), turned to 0 degrees
- moved J8 110.0 mm to (139.9, 95.6), turned to 0 degrees
- moved J9 109.9 mm to (139.9, 106.7), turned to 0 degrees
- moved J10 109.9 mm to (139.8, 117.9), turned to 0 degrees
- moved J3 94.4 mm to (93.0, 127.1)
- moved C2 85.4 mm to (88.0, 76.0), turned to -90 degrees
- moved JP3 70.3 mm to (107.5, 73.6)
- moved U1 70.1 mm to (96.9, 72.9), turned to 0 degrees
- moved JP2 67.1 mm to (107.5, 78.4)
- moved R10 64.7 mm to (131.6, 125.0), turned to 180 degrees
- moved JP1 64.5 mm to (107.5, 83.2)
- moved C3 61.3 mm to (94.0, 114.5)
- moved R9 59.1 mm to (131.6, 114.0), turned to 180 degrees
- moved R2 54.9 mm to (116.5, 115.6), turned to 90 degrees
- moved R8 54.2 mm to (131.6, 103.0), turned to 180 degrees
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Connections:
- C2 pad 1: +12V -> +3.3V
- C3 pad 1: +3.3V -> +12V
- J10 pad 2: /IO11 -> Net-(J10-Pin_2)
- J11 pad 2: /IO12 -> Net-(J11-Pin_2)
- J2 pad 1: /IO0 -> GND
- J2 pad 2: /IO1 -> +3.3V
- J2 pad 3: /IO2 -> Net-(U1-SDA)
- J2 pad 4: /IO3 -> Net-(U1-SCK)
- J3 pad 1: /IO8 -> +12V
- J3 pad 2: /IO9 -> GND
- J7 pad 2: /IO8 -> Net-(J7-Pin_2)
- J8 pad 2: /IO13 -> Net-(J8-Pin_2)
- J9 pad 2: /IO4 -> Net-(J9-Pin_2)
- R10 pad 1: /IO12 -> Net-(J11-Pin_2)
- R10 pad 2: GND -> Net-(U1-GPB7)
- R2 pad 1: +3.3V -> Net-(U1-SCK)
- R2 pad 2: Net-(U1-~{RESET}) -> Net-(JP4-B)
- R8 pad 1: /IO9 -> Net-(J9-Pin_2)
- R8 pad 2: GND -> Net-(U1-GPB5)
- R9 pad 1: /IO9 -> Net-(J10-Pin_2)
- R9 pad 2: Net-(Q4-G) -> Net-(U1-GPB6)
- U1 pad 1: /IO0 -> Net-(U1-GPB0)
- U1 pad 12: /SCK -> Net-(U1-SCK)
- U1 pad 13: /SDA -> Net-(U1-SDA)
- U1 pad 15: Net-(JP3-C) -> Net-(JP1-C)
- U1 pad 17: Net-(JP1-C) -> Net-(JP3-C)
- U1 pad 18: Net-(U1-~{RESET}) -> +3.3V
- U1 pad 2: /IO1 -> Net-(U1-GPB1)
- U1 pad 21: /IO8 -> Net-(U1-GPA0)
- U1 pad 22: /IO9 -> Net-(U1-GPA1)
- U1 pad 23: /IO10 -> Net-(U1-GPA2)
- U1 pad 24: /IO11 -> Net-(U1-GPA3)
- U1 pad 25: /IO12 -> Net-(U1-GPA4)
- U1 pad 26: /IO13 -> Net-(U1-GPA5)
- U1 pad 27: /IO11 -> Net-(U1-GPA6)
- U1 pad 28: /IO10 -> Net-(U1-GPA7)
- U1 pad 3: /IO2 -> Net-(U1-GPB2)
- U1 pad 4: /IO3 -> Net-(U1-GPB3)
- U1 pad 5: /IO4 -> Net-(U1-GPB4)
- U1 pad 6: /IO5 -> Net-(U1-GPB5)
- U1 pad 7: /IO13 -> Net-(U1-GPB6)
- U1 pad 8: /IO12 -> Net-(U1-GPB7)
Routing:
- net +3.3V: track 4.06 -> 122.4 mm
- net +12V: track 0.00 -> 91.7 mm
- net GND: track 3.98 -> 46.4 mm, vias 0 -> 3
- net Net-(U1-GPA7): track 0.00 -> 26.2 mm
- net Net-(U1-GPA6): track 0.00 -> 24.5 mm
- net Net-(U1-GPA5): track 0.00 -> 22.9 mm
- net Net-(U1-GPA4): track 0.00 -> 21.0 mm
- net Net-(U1-GPA3): track 0.00 -> 19.0 mm
- net Net-(U1-GPA2): track 0.00 -> 16.7 mm
- net Net-(J7-Pin_2): track 0.00 -> 16.4 mm
- net Net-(J11-Pin_2): track 0.00 -> 16.2 mm
- net Net-(J6-Pin_2): track 0.00 -> 16.2 mm
- net Net-(J5-Pin_2): track 0.00 -> 16.1 mm
- net Net-(J8-Pin_2): track 0.00 -> 16.0 mm
- net Net-(J4-Pin_2): track 0.00 -> 15.9 mm
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